File: Big Daddy-2025-04-11_172858/Big Daddy-2025-04-11_172858/TSAL.kicad_sch (KiCad schematic)
At the start: 20 parts, among them J1 TSSI_Grn I/O, J16 TSSI_Red I/O, Q2 BCP53, U5 LTV-817S, U6 ICM7555xB, U7 IS31LT3360

Commit message: updated lights
Parts:
- removed Q2: BCP53, Package_TO_SOT_SMD:SOT-223-3_TabPin2, symbol Transistor_BJT:BCP53
- removed R28: 1k, Resistor_SMD:R_0603_1608Metric_Pad0.98x0.95mm_HandSolder, symbol Device:R_US
- removed U5: LTV-817S, Package_DIP:SMDIP-4_W9.53mm, symbol Isolator:LTV-817S
- added Q2, Q5: RU1C002UN, symbol Transistor_FET:2N3819
- added R14: 2200, Resistor_THT:R_Axial_DIN0414_L11.9mm_D4.5mm_P15.24mm_Horizontal, symbol Device:R_US
- added U13: LTV-352T, Package_SO:SO-4_4.4x3.6mm_P2.54mm, symbol Isolator:LTV-352T
- R24: value 200k -> 300k; Digikey part number CF12JT39K0CT-ND -> 4491-MF2W300KFTTB-ND
Connections:
- net TSSI_Green is gone; now on net INT_12V: J1.2 (Pin_2)
- net TSSI_Red is gone; now on net INT_12V: J16.2 (Pin_2)
- net 555_OUT: now also Q2.2 (G)
- net GND: now also Q2.3 (S), Q5.3 (S), R14.2; no longer J1.1 (Pin_1), J16.1 (Pin_1)
- net HV-: now also U13.2
- net INT_12V: now also J16.1 (Pin_1), Q2.1 (D)
- net VDD: now also U13.4
- net at R24.2: now also U13.1
- new net: Q5.2 (G), R14.1, U13.3
- new net TSSI_Green_in: J1.1 (Pin_1), Q5.1 (D)
Other:
- note added: "RED TSI Blnky Light Requirement: 2-5 Hz, 50% duty cycle"
- moved on the sheet: J1, J16, R24

Commit message: footprints found for fets and Rs
Parts:
- Q2, Q5: footprint (none) -> Package_TO_SOT_SMD:SOT-323_SC-70
- R14: footprint Resistor_THT:R_Axial_DIN0414_L11.9mm_D4.5mm_P15.24mm_Horizontal -> Resistor_SMD:R_1206_3216Metric_Pad1.30x1.75mm_HandSolder; Digikey part number CF12JT39K0CT-ND -> 4463-TFA1206R2201J-T5CT-ND; Manufacturer_Part_Number CF12JT39K0 -> TFA1206R2201J-T5
- R24: footprint Resistor_THT:R_Axial_DIN0414_L11.9mm_D4.5mm_P15.24mm_Horizontal -> Resistor_THT:R_Axial_DIN0516_L15.5mm_D5.0mm_P30.48mm_Horizontal
Changed lines of the file:
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@@
 			)
 		)
-		(property "Footprint" ""
+		(property "Footprint" "Package_TO_SOT_SMD:SOT-323_SC-70"
 			(at 88.9 163.195 0)
 			(effects
@@
 			)
 		)
-		(property "Footprint" "Resistor_THT:R_Axial_DIN0414_L11.9mm_D4.5mm_P15.24mm_Horizontal"
+		(property "Footprint" "Resistor_SMD:R_1206_3216Metric_Pad1.30x1.75mm_HandSolder"
 			(at 79.756 114.554 90)
 			(effects
@@
 			)
 		)
-		(property "Datasheet" "https://www.seielect.com/catalog/sei-cf_cfm.pdf"
+		(property "Datasheet" "https://www.thin-film.com/wp-content/uploads/2023/03/TFA-Series-TFT-DMS-341-1.pdf"
 			(at 78.74 114.3 0)
 			(effects
@@
 			)
 		)
-		(property "Digikey part number" "CF12JT39K0CT-ND"
+		(property "Digikey part number" "4463-TFA1206R2201J-T5CT-ND"
 			(at 78.74 114.3 0)
 			(effects
@@
 			)
 		)
-		(property "Manufacturer_Part_Number" "CF12JT39K0"
+		(property "Manufacturer_Part_Number" "TFA1206R2201J-T5"
 			(at 78.74 114.3 0)
 			(effects
@@
 			)
 		)
-		(property "Footprint" "Resistor_THT:R_Axial_DIN0414_L11.9mm_D4.5mm_P15.24mm_Horizontal"
+		(property "Footprint" "Resistor_THT:R_Axial_DIN0516_L15.5mm_D5.0mm_P30.48mm_Horizontal"
 			(at 55.626 90.424 90)
 			(effects
@@
 			)
 		)
-		(property "Footprint" ""
+		(property "Footprint" "Package_TO_SOT_SMD:SOT-323_SC-70"
 			(at 223.52 158.115 0)
 			(effects
