File: Big Daddy-2025-04-11_172858/Big Daddy-2025-04-11_172858/Big Daddy.kicad_pcb (KiCad board)
At the start: 4 copper layers, 245.7 x 126.7 mm, 120 parts, among them J10 Conn_01x02, J11 Conn_01x23, J12 Conn_01x14, J13 Conn_01x14, J14 BMS Button, J15 Conn_01x02, J2 IMD Button, J3 HV+, J4 HV-, J5 GND, J6 HV+, J7 HV-, J8 Conn_01x14, J9 Conn_01x08, K1 T9VV1K15-12S, K2 G5V-1, K3 G5V-2, K4 J107, K5 G5V-1, Q1 2N7002, Q2 BCP53, Q3 IXFH34N65X2, Q4 IXFH34N65X2, U1 MAX33054EASA+T, U10 TLP184, U14 LM317_TO-263, U2 ESP32-S3-DevKitC, U3 ESP32-S3-DevKitC, U4 LT1528CQ#PBF, U5 LTV-817S, U6 ICM7555xB, U7 IS31LT3360, U8 Vicor_AERO, U9 LTV-817S

Commit message: Rerouted PCB
Parts:
- removed C12: 100uF, Capacitor_THT:CP_Radial_D10.0mm_P5.00mm
- removed C13, C18, C19, C20: .1uF, Capacitor_SMD:C_0603_1608Metric_Pad1.08x0.95mm_HandSolder
- removed D10, D11: SS16, Diode_SMD:D_SMA
- removed D9: D_Zener, Diode_SMD:D_SOD-123
- removed J9: Conn_01x08, AERO_Footprints:TE_1-776280-1_8pin_Horizontal
- removed L1: 47uH, Inductor_SMD:L_0603_1608Metric_Pad1.05x0.95mm_HandSolder
- removed Q3, Q4: IXFH34N65X2, PCM_Package_TO_SOT_THT_AKL:TO-247-3_Vertical_GDS
- removed R26, R29: 10k, Resistor_SMD:R_0603_1608Metric_Pad0.98x0.95mm_HandSolder
- removed R28: 1k, Resistor_SMD:R_0603_1608Metric_Pad0.98x0.95mm_HandSolder
- removed R30: 0.15, Resistor_SMD:R_0603_1608Metric_Pad0.98x0.95mm_HandSolder
- removed R31: 100, Resistor_SMD:R_1206_3216Metric_Pad1.30x1.75mm_HandSolder
- removed R34: .2, Resistor_SMD:R_0805_2012Metric_Pad1.20x1.40mm_HandSolder
- removed R41: 2.2k, Resistor_SMD:R_0603_1608Metric_Pad0.98x0.95mm_HandSolder
- removed R42: 2.4k, Resistor_SMD:R_0603_1608Metric_Pad0.98x0.95mm_HandSolder
- removed R43: 240, Resistor_SMD:R_0603_1608Metric_Pad0.98x0.95mm_HandSolder
- removed U14: LM317_TO-263, Package_TO_SOT_SMD:TO-263-2
- removed U5: LTV-817S, Package_DIP:SMDIP-4_W9.53mm
- removed U7: IS31LT3360, Package_TO_SOT_SMD:SOT-89-5
- added J1: TSSI_Grn I/O, Connector_Hirose:Hirose_DF63R-2P-3.96DSA_1x02_P3.96mm_Vertical, F.Cu at (210.8, 168.7)
- added J16: TSSI_Red I/O, Connector_Hirose:Hirose_DF63R-2P-3.96DSA_1x02_P3.96mm_Vertical, F.Cu at (200.2, 168.7)
- added J17: Conn_01x14, AERO_Footprints:TE_1-776266-1_14pin_Horizontal, F.Cu at (170.8, 178.4)
- added Q5: RU1C002UN, Package_TO_SOT_SMD:SOT-323_SC-70, B.Cu at (167.6, 165.6)
- added R14: 2200, Resistor_SMD:R_1206_3216Metric_Pad1.30x1.75mm_HandSolder, B.Cu at (143.3, 152.9)
- added U13: LTV-352T, Package_SO:SO-4_4.4x3.6mm_P2.54mm, B.Cu at (134.6, 154.4)
- Q2: value BCP53 -> RU1C002UN; footprint Package_TO_SOT_SMD:SOT-223-3_TabPin2 -> Package_TO_SOT_SMD:SOT-323_SC-70
- R16: value 5.97k -> 2.2k
- R24: value 39k -> 300k; footprint Resistor_THT:R_Axial_DIN0414_L11.9mm_D4.5mm_P15.24mm_Horizontal -> Resistor_THT:R_Axial_DIN0516_L15.5mm_D5.0mm_P30.48mm_Horizontal
- R27: value 15k -> 24k
- moved Q2 6.25 mm to (168.3, 157.6), turned to 90 degrees
Connections:
- net +12V renamed Net-(F1-Pad1)
- C4 pad 1: INT_12V -> /Connectors/TSSI_Green_out
- D12 pad 1: Net-(D12-K) -> /Latching/BMS_Switch
- D3 pad 1: INT_12V -> /Connectors/TSSI_Green_out
- F1 pad 2: INT_12V -> /Connectors/TSSI_Green_out
- F10 pad 2: /Connectors/SSOK -> /Connectors/TSV
- J12 pad 6: /Connectors/RTD_LED -> /Connectors/DRIVE_MODE_LED
- J13 pad 6: /Connectors/PUMP_TEMP_OUT -> /Connectors/PUMP_TEMP_IN
- J14 pad 1: INT_12V -> /Connectors/TSSI_Green_out
- J2 pad 2: INT_12V -> /Connectors/TSSI_Green_out
- K1 pad 3: /Fusing/12_prefuse -> /Fusing/Vicor_In
- K2 pad 10: INT_12V -> /Connectors/TSSI_Green_out
- Q2 pad 1: Net-(Q2-B) -> /Connectors/TSSI_Red_in
- Q2 pad 2: /Connectors/TSAL_PWR -> /High Voltage/TSAL/555_OUT
- Q2 pad 3: INT_12V -> GND
- R16 pad 1: Net-(D12-K) -> /Latching/BMS_Switch
- R16 pad 2: /Latching/BMS_IND -> /Connectors/BMS_FAULT_SIG
- R25 pad 1: /High Voltage/TSAL/HV_ON -> /High Voltage/TSSI_Fault
- R27 pad 1: /High Voltage/TSAL/555_OUT -> VDD
- R7 pad 1: /Connectors/RTD_LED -> /Connectors/DRIVE_MODE_LED
- U2 pad 13: unconnected-(U2-GPIO3/ADC1_CH2-Pad13) -> /High Voltage/TSSI_Fault
- U2 pad 32: /Microcontrolller/SCL -> unconnected-(U2-GPIO35-Pad32)
- U2 pad 33: /Microcontrolller/SDA -> unconnected-(U2-GPIO36-Pad33)
- U2 pad 40: /Connectors/PUMP_TEMP_OUT -> /Connectors/PUMP_TEMP_IN
- U2 pad 8: /Latching/BMS_IND -> /Connectors/BMS_FAULT_SIG
- U3 pad 42: /Microcontrolller/Core_RX -> unconnected-(U3-GPIO44/U0RXD-Pad42)
- U3 pad 43: /Microcontrolller/Core_TX -> unconnected-(U3-GPIO43/U0TXD-Pad43)
- U4 pad 5: INT_12V -> /Connectors/TSSI_Green_out
- U6 pad 4: /High Voltage/TSAL/HV_ON -> /High Voltage/TSSI_Fault
- U6 pad 7: Net-(U6-DIS) -> VDD
Routing:
- net /High Voltage/TSSI_Fault: track 0.00 -> 141.2 mm, vias 0 -> 3
- net INT_12V: track 104.4 -> 0.00 mm, vias 6 -> 0
- net /Connectors/DRIVE_MODE_LED: track 37.8 -> 121.3 mm
- net /Connectors/PUMP_TEMP_OUT: track 83.4 -> 0.00 mm, vias 1 -> 0
- net /Connectors/BMS_FAULT_SIG: track 113.5 -> 191.2 mm
- net /Connectors/TSSI_Green_out: track 0.00 -> 73.4 mm
- net /Latching/BMS_IND: track 72.7 -> 0.00 mm
- net /Connectors/RTD_LED: track 67.9 -> 0.00 mm
- net /Connectors/TSSI_Green_in: track 0.00 -> 61.2 mm
- net /Connectors/TSAL_PWR: track 56.3 -> 0.00 mm
- net /Connectors/TSSI_Red_in: track 0.00 -> 52.8 mm, vias 0 -> 2
- net Net-(Q5-G): track 0.00 -> 38.7 mm, vias 0 -> 4
- net /Connectors/TSV: track 0.00 -> 34.3 mm
- net /Connectors/TSAL_GND: track 34.2 -> 0.00 mm
- net /Connectors/PUMP_TEMP_IN: track 79.2 -> 109.7 mm, vias 1 -> 2
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- added copper zone on In1.Cu, net /Connectors/TSSI_Green_out
- removed copper zone on B.Cu, net /Fusing/12_prefuse
- removed copper zone on F.Cu, net /Fusing/12_prefuse
- removed copper zone on In1.Cu, net INT_12V
Other:
- board size 245.7 x 126.7 mm -> 247.4 x 126.7 mm
