File: Big Daddy-2025-04-11_172858/Big Daddy-2025-04-11_172858/Big Daddy.kicad_sch (KiCad schematic)
At the start: 0 parts

Commit message: Rerouted PCB
Connections:
- no-connect marks 0 -> 1
Other:
- sheet Connectors ports: added none; removed FAN_LED, PUMP_LED
- sheet Microcontrolller ports: added none; removed FAN_LED, PUMP_LED
Changed lines of the file:
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@@
 	)
 	(junction
+		(at 80.01 111.76)
+		(diameter 0)
+		(color 0 0 0 0)
+	)
+	(junction
 		(at 85.5161 169.672)
 		(diameter 0)
@@
 		(color 0 0 0 0)
 	)
+	(no_connect
+		(at 227.33 99.06)
+	)
+	(wire
+		(pts
+			(xy 224.282 99.06) (xy 227.33 99.06)
+		)
+		(stroke
+			(width 0)
+			(type default)
+		)
+	)
 	(wire
 		(pts
@@
 	(wire
 		(pts
-			(xy 75.692 111.76) (xy 91.948 111.76)
+			(xy 75.692 111.76) (xy 80.01 111.76)
 		)
 		(stroke
@@
 	(wire
 		(pts
-			(xy 145.034 80.01) (xy 189.484 80.01)
-		)
-		(stroke
-			(width 0)
-			(type default)
-		)
-	)
-	(wire
-		(pts
 			(xy 145.034 35.814) (xy 166.624 35.814)
 		)
@@
 	(wire
 		(pts
+			(xy 74.93 36.83) (xy 80.01 36.83)
+		)
+		(stroke
+			(width 0)
+			(type default)
+		)
+	)
+	(wire
+		(pts
 			(xy 29.21 83.312) (xy 29.21 146.05)
 		)
@@
 	(wire
 		(pts
+			(xy 80.01 36.83) (xy 80.01 111.76)
+		)
+		(stroke
+			(width 0)
+			(type default)
+		)
+	)
+	(wire
+		(pts
 			(xy 199.644 96.266) (xy 199.644 91.186)
 		)
@@
 	(wire
 		(pts
-			(xy 189.484 80.01) (xy 189.484 74.93)
-		)
-		(stroke
-			(width 0)
-			(type default)
-		)
-	)
-	(wire
-		(pts
 			(xy 238.76 163.322) (xy 238.76 114.046)
 		)
@@
 	(wire
 		(pts
-			(xy 189.484 74.93) (xy 190.754 74.93)
+			(xy 164.084 27.686) (xy 190.754 27.686)
 		)
 		(stroke
@@
 	(wire
 		(pts
-			(xy 164.084 27.686) (xy 190.754 27.686)
+			(xy 76.2 147.32) (xy 91.948 147.32)
 		)
 		(stroke
@@
 	(wire
 		(pts
-			(xy 76.2 147.32) (xy 91.948 147.32)
+			(xy 80.01 111.76) (xy 91.948 111.76)
 		)
 		(stroke
@@
 			)
 		)
-		(pin "FAN_LED" input
-			(at 190.754 77.978 180)
-			(effects
-				(font
-					(size 1.27 1.27)
-				)
-				(justify left)
-			)
-		)
-		(pin "PUMP_LED" input
-			(at 190.754 74.93 180)
-			(effects
-				(font
-					(size 1.27 1.27)
-				)
-				(justify left)
-			)
-		)
 		(pin "BMS_Fault" input
 			(at 224.282 112.522 0)
@@
 			)
 		)
-		(pin "PUMP_LED" input
-			(at 145.034 80.01 0)
-			(effects
-				(font
-					(size 1.27 1.27)
-				)
-				(justify right)
-			)
-		)
 		(pin "CAN_L" output
 			(at 145.034 130.048 0)
@@
 			(effects
 				(font
-					(size 1.27 1.27)
-				)
-				(justify right)
-			)
-		)
-		(pin "FAN_LED" input
-			(at 145.034 83.058 0)
-			(effects
-				(font
