File: Big Daddy-2025-04-11_172858/Big Daddy-2025-04-11_172858/Cooling.kicad_sch (KiCad schematic)
At the start: 7 parts, among them K4 J107, K5 G5V-1

Commit message: Rerouted PCB
Connections:
- no-connect marks 0 -> 1
Changed lines of the file:
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@@
 		(color 0 0 0 0)
+	)
+	(no_connect
+		(at 137.16 81.28)
 	)
 	(polyline
