File: Big Daddy-2025-04-11_172858/Big Daddy-2025-04-11_172858/Fusing.kicad_sch (KiCad schematic)
At the start: 17 parts, among them K1 T9VV1K15-12S, U4 LT1528CQ#PBF

Commit message: Rerouted PCB
Connections:
- net +12V: no longer names the net of F1.1, F2.1, F3.1, F4.1, F5.1, F6.1, F7.1, K1.4
Changed lines of the file:
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@@
+	)
+	(junction
+		(at 203.2 32.1393)
+		(diameter 0)
+		(color 0 0 0 0)
 	)
 	(junction
@@
 	)
 	(junction
+		(at 71.628 35.814)
+		(diameter 0)
+		(color 0 0 0 0)
+	)
+	(junction
 		(at 237.744 140.462)
 		(diameter 0)
@@
 	(wire
 		(pts
+			(xy 71.628 35.814) (xy 71.628 32.1393)
+		)
+		(stroke
+			(width 0)
+			(type default)
+		)
+	)
+	(wire
+		(pts
 			(xy 53.594 57.658) (xy 46.99 57.658)
 		)
@@
 	(wire
 		(pts
-			(xy 203.2 32.004) (xy 203.2 40.894)
+			(xy 203.2 32.004) (xy 203.2 32.1393)
 		)
 		(stroke
@@
 	(wire
 		(pts
+			(xy 203.2 32.1393) (xy 203.2 40.894)
+		)
+		(stroke
+			(width 0)
+			(type default)
+		)
+	)
+	(wire
+		(pts
 			(xy 182.88 122.682) (xy 189.992 122.682)
 		)
@@
 		)
 	)
+	(wire
+		(pts
+			(xy 71.628 32.1393) (xy 203.2 32.1393)
+		)
+		(stroke
+			(width 0)
+			(type default)
+		)
+	)
 	(polyline
 		(pts
@@
 		(pts
 			(xy 46.99 45.72) (xy 46.99 45.974)
+		)
+		(stroke
+			(width 0)
+			(type default)
+		)
+	)
+	(wire
+		(pts
+			(xy 71.628 35.8489) (xy 71.628 35.814)
 		)
 		(stroke
@@
 	)
 	(symbol
-		(lib_id "power:+12V")
-		(at 203.2 32.004 0)
-		(mirror y)
-		(unit 1)
-		(exclude_from_sim no)
-		(in_bom yes)
-		(on_board yes)
-		(dnp no)
-		(property "Reference" "#PWR025"
-			(at 203.2 35.814 0)
-			(effects
-				(font
-					(size 1.27 1.27)
-				)
-				(hide yes)
-			)
-		)
-		(property "Value" "+12V"
-			(at 202.819 27.6098 0)
-			(effects
-				(font
-					(size 1.27 1.27)
-				)
-			)
-		)
-		(property "Footprint" ""
-			(at 203.2 32.004 0)
-			(effects
-				(font
-					(size 1.27 1.27)
-				)
-				(hide yes)
-			)
-		)
-		(property "Datasheet" ""
-			(at 203.2 32.004 0)
-			(effects
-				(font
-					(size 1.27 1.27)
-				)
-				(hide yes)
-			)
-		)
-		(property "Description" ""
-			(at 203.2 32.004 0)
-			(effects
-				(font
-					(size 1.27 1.27)
-				)
-				(hide yes)
-			)
-		)
-		(pin "1"
-		)
-		(instances
-			(project "Big Daddy"
-				(path "/e63e39d7-6ac0-4ffd-8aa3-1841a4541b55/9c1412ff-15e3-4ef7-9c9c-e6f8f725cc08"
-					(reference "#PWR025")
-					(unit 1)
-				)
-			)
-		)
-	)
-	(symbol
 		(lib_id "power:GND")
 		(at 218.44 141.478 0)
@@
 					(unit 1)
 				)
-			)
-		)
-	)
-	(symbol
-		(lib_id "power:+12V")
-		(at 71.628 35.814 0)
-		(mirror y)
-		(unit 1)
-		(exclude_from_sim no)
-		(in_bom yes)
-		(on_board yes)
-		(dnp no)
-		(property "Reference" "#PWR024"
-			(at 71.628 39.624 0)
-			(effects
-				(font
-					(size 1.27 1.27)
-				)
-				(hide yes)
-			)
-		)
-		(property "Value" "+12V"
-			(at 71.247 31.4198 0)
-			(effects
-				(font
-					(size 1.27 1.27)
-				)
-			)
-		)
-		(property "Footprint" ""
-			(at 71.628 35.814 0)
-			(effects
-				(font
-					(size 1.27 1.27)
-				)
-				(hide yes)
-			)
-		)
-		(property "Datasheet" ""
-			(at 71.628 35.814 0)
-			(effects
-				(font
-					(size 1.27 1.27)
-				)
-				(hide yes)
-			)
-		)
-		(property "Description" ""
-			(at 71.628 35.814 0)
-			(effects
-				(font
-					(size 1.27 1.27)
-				)
-				(hide yes)
-			)
-		)
-		(pin "1"
-		)
-		(instances
-			(project "Big Daddy"
-				(path "/e63e39d7-6ac0-4ffd-8aa3-1841a4541b55/9c1412ff-15e3-4ef7-9c9c-e6f8f725cc08"
-					(reference "#PWR024")
-					(unit 1)
-				)
