File: Big Daddy-2025-04-11_172858/Big Daddy-2025-04-11_172858/Micro.kicad_sch (KiCad schematic)
At the start: 22 parts, among them Q1 2N7002, U1 MAX33054EASA+T, U2 ESP32-S3-DevKitC, U3 ESP32-S3-DevKitC

Commit message: Rerouted PCB
Connections:
- net Core_RX: no longer names the net of U3.42 (GPIO44/U0RXD)
- net Core_TX: no longer names the net of U3.43 (GPIO43/U0TXD)
- net SCL: no longer names the net of U2.32 (GPIO35)
- net SDA: no longer names the net of U2.33 (GPIO36)
- no-connect marks 18 -> 22
Other:
- note added: "Core_RX"
- note added: "Core_TX"
- note added: "SCL"
- note added: "SDA"
Changed lines of the file:
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@@
+		)
+	)
+	(text "SCL"
+		(exclude_from_sim no)
+		(at 104.394 90.424 0)
+		(effects
+			(font
+				(size 1.27 1.27)
+			)
+		)
+	)
+	(text "Core_TX"
+		(exclude_from_sim no)
+		(at 231.902 61.468 0)
+		(effects
+			(font
+				(size 1.27 1.27)
+			)
+		)
+	)
+	(text "Core_RX"
+		(exclude_from_sim no)
+		(at 232.156 63.5 0)
+		(effects
+			(font
+				(size 1.27 1.27)
+			)
 		)
 	)
@@
 		)
 	)
+	(text "SDA"
+		(exclude_from_sim no)
+		(at 104.394 87.884 0)
+		(effects
+			(font
+				(size 1.27 1.27)
+			)
+		)
+	)
 	(text "Telemetry Core"
 		(exclude_from_sim no)
@@
 	)
 	(no_connect
+		(at 101.6 87.63)
+	)
+	(no_connect
 		(at 226.822 73.66)
 	)
@@
 	)
 	(no_connect
+		(at 226.822 63.5)
+	)
+	(no_connect
 		(at 226.822 101.6)
 	)
@@
 	)
 	(no_connect
+		(at 226.822 60.96)
+	)
+	(no_connect
 		(at 176.022 81.28)
 	)
@@
 	)
 	(no_connect
+		(at 101.6 90.17)
+	)
+	(no_connect
 		(at 101.6 62.23)
 	)
@@
 		)
 	)
-	(wire
-		(pts
-			(xy 105.664 90.17) (xy 101.6 90.17)
-		)
-		(stroke
-			(width 0)
-			(type default)
-		)
-	)
 	(polyline
 		(pts
@@
 		)
 	)
-	(wire
-		(pts
-			(xy 238.506 60.96) (xy 226.822 60.96)
-		)
-		(stroke
-			(width 0)
-			(type default)
-		)
-	)
 	(polyline
 		(pts
@@
 	(wire
 		(pts
-			(xy 105.664 87.63) (xy 101.6 87.63)
-		)
-		(stroke
-			(width 0)
-			(type default)
-		)
-	)
-	(wire
-		(pts
 			(xy 134.62 187.96) (xy 134.62 191.262)
 		)
@@
 		(pts
 			(xy 43.942 95.25) (xy 50.8 95.25)
-		)
-		(stroke
-			(width 0)
-			(type default)
-		)
-	)
-	(wire
-		(pts
-			(xy 226.822 63.5) (xy 238.506 63.5)
 		)
 		(stroke
@@
 		)
 	)
-	(label "Core_RX"
-		(at 238.506 63.5 180)
-		(effects
-			(font
-				(size 1.27 1.27)
-			)
-			(justify right bottom)
-		)
-	)
-	(label "SCL"
-		(at 105.664 90.17 180)
-		(effects
-			(font
-				(size 1.27 1.27)
-			)
-			(justify right bottom)
-		)
-	)
 	(label "CAN_TX"
 		(at 101.092 74.93 0)
@@
 		)
 	)
-	(label "SDA"
-		(at 105.664 87.63 180)
-		(effects
-			(font
-				(size 1.27 1.27)
-			)
-			(justify right bottom)
-		)
-	)
 	(label "CAN_RX"
 		(at 17.78 172.212 0)
@@
 		)
 	)
-	(label "Core_TX"
-		(at 238.506 60.96 180)
-		(effects
-			(font
-				(size 1.27 1.27)
-			)
-			(justify right bottom)
-		)
-	)
